Commit message: map can be generated, but frame:map can't be found

File: src/my_package/resource/my_robot.urdf (robot description, URDF)
Before this commit: robot My robot, 0 links, 0 joints
Links:
- added link accelerometer
- added link base_link; collision cylinder length=0.08 radius=0.045; visual cylinder length=0.08 radius=0.045
- added link gyro
- added link inertial_unit
- added link left wheel; collision cylinder length=0.01 radius=0.025; visual cylinder length=0.01 radius=0.025
- added link lidar
- added link right wheel; collision cylinder length=0.01 radius=0.025; visual cylinder length=0.01 radius=0.025
Joints:
- added joint base_link_accelerometer_joint: type fixed, parent base_link, child accelerometer, origin xyz=0 0 0.1 rpy=0 0 0
- added joint base_link_gyro_joint: type fixed, parent base_link, child gyro, origin xyz=0 0 0.1 rpy=0 0 0
- added joint base_link_inertial_unit_joint: type fixed, parent base_link, child inertial_unit, origin xyz=0 0 0.1 rpy=0 0 0
- added joint base_link_lidar_joint: type fixed, parent base_link, child lidar, origin xyz=0 0 0.1 rpy=0 0 0
- added joint left wheel motor: type continuous, parent base_link, child left wheel, origin xyz=0 -0.045 0.025 rpy=0 0 0, axis 0 1 0, limit effort=10 velocity=10
- added joint right wheel motor: type continuous, parent base_link, child right wheel, origin xyz=0 0 0.025 rpy=0 0.000001 0, axis 0 1 0, limit effort=10 velocity=10
